File: choc/korris/korris.kicad_pcb (KiCad board)
At the start: 2 copper layers, 124 parts, among them J1 AudioJack4, J2 USB_C, J3 AudioJack4, K1 KEYSW, K10 KEYSW, K11 KEYSW, K12 KEYSW, K13 KEYSW, K14 KEYSW, K15 KEYSW, K16 KEYSW, K17 KEYSW, K18 KEYSW, K19 KEYSW, K2 KEYSW, K20 KEYSW, K21 KEYSW, K22 KEYSW, K23 KEYSW, K24 KEYSW, K25 KEYSW, K26 KEYSW, K27 KEYSW, K28 KEYSW, K29 KEYSW, K3 KEYSW, K30 KEYSW, K31 KEYSW, K32 KEYSW, K33 KEYSW, K34 KEYSW, K35 KEYSW, K36 KEYSW, K37 KEYSW, K38 KEYSW, K39 KEYSW, K4 KEYSW, K40 KEYSW, K41 KEYSW, K42 KEYSW, K43 KEYSW, K44 KEYSW, K5 KEYSW, K6 KEYSW, K7 KEYSW, K8 KEYSW, K9 KEYSW, Q1 MMBT3904, SW1 SW_Push, U1 XC6206PxxxMR, U2 MCP23017_SO, U3 STM32F072CBUx, U4 SRV05-4

Commit message: add outline for choc layout
Parts:
- added SW2: Rotary_Encoder_Switch, Keebio-Parts:RotaryEncoder_EC11, F.Cu at (-37.3, 6.25)
- added SW3: Rotary_Encoder_Switch, Keebio-Parts:RotaryEncoder_EC11, F.Cu at (27.3, 3.34)
- J1, J3: footprint Keebio-Parts:TRRS-PJ-320A -> hy-keebs:TRRS-PJ-320Atrrs
- J2: footprint Connector_USB:USB_C_Receptacle_HRO_TYPE-C-31-M-12 -> hy-keebs:USB_C_HRO_TYPE-C-31-M-12
- moved C4 299.7 mm to (41.9, -29.1), turned to 270 degrees
- moved R8 274.8 mm to (37.6, -78.9), turned to 90 degrees
- moved C9 240.6 mm to (112.7, -44.7), turned to 90 degrees
- moved C2 236.7 mm to (112.7, -40.0), turned to 270 degrees
- moved C12 222.1 mm to (124.2, -40.8), turned to 270 degrees
- moved R10 206.3 mm to (151.5, -57.6)
- moved R1 195.4 mm to (116.8, -46.9), turned to 90 degrees
- moved C8 188.5 mm to (152.4, -35.2), turned to 180 degrees
- moved R2 186.5 mm to (122.8, -44.9)
- moved R7 179.9 mm to (37.6, -75.7), turned to 270 degrees
- moved C3 143.6 mm to (40.1, -29.0), turned to 270 degrees
- moved SW1 120.9 mm to (119.8, -52.1), turned to 270 degrees
- moved D45 110.3 mm to (120.0, -47.0)
- moved C6 106.1 mm to (124.2, -36.8), turned to 90 degrees
- moved U1 100.7 mm to (48.1, -28.7)
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Connections:
- U2 pad 1: (no net) -> /row1,0
- U2 pad 2: (no net) -> /row1,1
- U2 pad 21: (no net) -> /col6
- U2 pad 22: (no net) -> /col7
- U2 pad 23: (no net) -> /col8
- U2 pad 24: (no net) -> /col9
- U2 pad 25: (no net) -> /col10
- U2 pad 26: (no net) -> /col11
- U2 pad 3: (no net) -> /row1,2
- U2 pad 4: (no net) -> /row1,3
- U3 pad 21: (no net) -> i2c_scl
- U3 pad 22: (no net) -> i2c_sda
- U3 pad 34: (no net) -> /col5
- U3 pad 37: (no net) -> /col4
- U3 pad 38: (no net) -> /col3
- U3 pad 39: (no net) -> /col2
- U3 pad 40: (no net) -> /col1
- U3 pad 44: (no net) -> BOOT0
- U3 pad 45: (no net) -> /col0
- U3 pad 7: (no net) -> NRST
Other:
- board outline added: 264 x 87.1 mm

Commit message: routed left half
Parts:
- U3: footprint Package_DFN_QFN:QFN-48-1EP_7x7mm_P0.5mm_EP5.6x5.6mm -> breakout_pins:Dual_MCU_QFP_QFN_48_with_breakout_pins
- moved R3 25.2 mm to (113.1, -56.7)
- moved C2 16.9 mm to (115.0, -56.7)
- moved SW1 15.6 mm to (128.9, -39.5), turned to 90 degrees
- moved R4 10.3 mm to (115.0, -60.7)
- moved Q1 10.3 mm to (112.1, -60.4)
- moved R5 10.0 mm to (116.9, -56.7)
- moved D45 9.48 mm to (120.7, -56.5), turned to 90 degrees
- moved F1 8.34 mm to (39.8, -24.2), turned to 180 degrees
- moved C6 7.93 mm to (127.0, -44.2)
- moved C7 7.91 mm to (152.5, -50.0)
- moved R10 7.91 mm to (149.0, -50.1)
- moved R9 7.91 mm to (145.3, -50.1)
- moved U2 7.91 mm to (147.6, -38.4)
- moved R2 7.80 mm to (119.0, -51.7), turned to 90 degrees
- moved R6 7.55 mm to (155.0, -31.2), turned to 270 degrees
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Connections:
- U3 pad 10: (no net) -> Net-(U3-Pad10)
- U3 pad 11: (no net) -> Net-(U3-Pad11)
- U3 pad 13: (no net) -> Net-(U3-Pad13)
- U3 pad 14: (no net) -> Net-(U3-Pad14)
- U3 pad 15: (no net) -> Net-(U3-Pad15)
- U3 pad 16: (no net) -> Net-(U3-Pad16)
- U3 pad 17: (no net) -> Net-(U3-Pad17)
- U3 pad 18: (no net) -> Net-(U3-Pad18)
- U3 pad 19: (no net) -> Net-(U3-Pad19)
- U3 pad 2: (no net) -> Net-(U3-Pad2)
- U3 pad 20: (no net) -> Net-(U3-Pad20)
- U3 pad 25: (no net) -> Net-(U3-Pad25)
- U3 pad 26: (no net) -> Net-(U3-Pad26)
- U3 pad 27: (no net) -> Net-(U3-Pad27)
- U3 pad 28: (no net) -> Net-(U3-Pad28)
- U3 pad 29: (no net) -> Net-(U3-Pad29)
- U3 pad 3: (no net) -> Net-(U3-Pad3)
- U3 pad 30: (no net) -> Net-(U3-Pad30)
- U3 pad 31: (no net) -> Net-(U3-Pad31)
- U3 pad 4: (no net) -> Net-(U3-Pad4)
- U3 pad 41: /row0,2 -> /row0,0
- U3 pad 43: /row0,0 -> /row0,2
- U3 pad 46: (no net) -> Net-(U3-Pad46)
- U3 pad 5: (no net) -> Net-(U3-Pad5)
- U3 pad 6: (no net) -> Net-(U3-Pad6)
Routing:
- net /D+: track 0.00 -> 229.2 mm, vias 0 -> 1
- net /D-: track 0.00 -> 225.5 mm, vias 0 -> 1
- net +3V3: track 0.00 -> 210.9 mm, vias 0 -> 7
- net /col2: track 0.00 -> 177.8 mm, vias 0 -> 1
- net /col1: track 0.00 -> 175.6 mm, vias 0 -> 1
- net /row0,0: track 0.00 -> 167.6 mm, vias 0 -> 4
- net /col3: track 0.00 -> 162.4 mm, vias 0 -> 1
- net /col0: track 0.00 -> 152.6 mm
- net /col4: track 0.00 -> 142.3 mm, vias 0 -> 2
- net /row0,1: track 0.00 -> 136.5 mm
- net /row0,2: track 0.00 -> 130.9 mm, vias 0 -> 2
- net /col5: track 0.00 -> 124.0 mm, vias 0 -> 2
- net GND: track 0.00 -> 92.5 mm, vias 0 -> 11
- net /row0,3: track 0.00 -> 73.7 mm, vias 0 -> 1
- net /col6: track 0.00 -> 72.8 mm
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- added copper zone on B.Cu, net GND
- added copper zone on F.Cu, net GND
Other:
- outline, holes or cut-outs redrawn
- net class power added: clearance 0.2, trace_width 0.3, via_dia 0.8, via_drill 0.4

Commit message: add unicorn design
Parts:
- added REF**: mouse-bite-2mm-slot-with-space-for-track, panelization:mouse-bite-2mm-slot-with-space-for-track, F.Cu at (132.8, -60.4)
- added REF**: mouse-bite-2mm-slot-with-space-for-track, panelization:mouse-bite-2mm-slot-with-space-for-track, F.Cu at (132.8, -25.9)
- moved C7 17.1 mm to (141.1, -37.2), turned to 270 degrees
- moved C8 15.8 mm to (139.4, -37.2)
- moved R10 9.10 mm to (140.2, -48.0), turned to 180 degrees
- moved R6 8.46 mm to (155.4, -39.7), turned to 90 degrees
- moved U2 6.63 mm to (148.7, -45.0), turned to 0 degrees
- moved R9 6.37 mm to (140.2, -46.3)
Routing:
- net /row1,0: track 0.00 -> 138.4 mm
- net /row1,1: track 0.00 -> 132.9 mm
- net /row1,2: track 0.00 -> 129.9 mm
- net /col11: track 38.9 -> 151.4 mm
- net /row1,3: track 0.00 -> 101.3 mm
- net /col10: track 39.6 -> 138.4 mm
- net VDD: track 0.00 -> 77.4 mm
- net /col9: track 64.6 -> 133.6 mm
- net /col8: track 67.3 -> 131.2 mm
- net /col7: track 65.6 -> 109.1 mm
- net i2c_sda_right: track 0.00 -> 23.4 mm
- net /col6: track 72.8 -> 95.0 mm
- net Net-(J2-PadS1): track 0.00 -> 21.6 mm
- net i2c_scl_right: track 0.00 -> 19.2 mm
- net GND: track 92.5 -> 75.2 mm, vias 11 -> 16
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