File: unicorn-mx/unicorn/unicorn.sch (KiCad schematic (older format))
At the start: 118 parts, among them J2 USB_C, K1 KEYSW, K10 KEYSW, K11 KEYSW, K12 KEYSW, K13 KEYSW, K14 KEYSW, K15 KEYSW, K16 KEYSW, K17 KEYSW, K18 KEYSW, K19 KEYSW, K2 KEYSW, K20 KEYSW, K21 KEYSW, K22 KEYSW, K23 KEYSW, K24 KEYSW, K25 KEYSW, K26 KEYSW, K27 KEYSW, K28 KEYSW, K29 KEYSW, K3 KEYSW, K30 KEYSW, K31 KEYSW, K32 KEYSW, K33 KEYSW, K34 KEYSW, K35 KEYSW, K36 KEYSW, K37 KEYSW, K38 KEYSW, K39 KEYSW, K4 KEYSW, K40 KEYSW, K41 KEYSW, K42 KEYSW, K43 KEYSW, K44 KEYSW, K5 KEYSW, K6 KEYSW, K7 KEYSW, K8 KEYSW, K9 KEYSW, Q1 MMBT3904, SW1 SW_Push, SW2 Rotary_Encoder_Switch, SW3 Rotary_Encoder_Switch, U1 XC6206PxxxMR, U3 STM32F072CBUx, U4 SRV05-4

Commit message: add 3d models, add oled
Parts:
- added OL?: OLED, symbol kbd:OLED
Connections:
- net +3V3: now also OL?.3 (VCC)
- net GND: now also OL?.4 (GND)
- net i2c_scl: now also OL?.2 (SCL)
- net i2c_sda: now also OL?.1 (SDA)
Changed lines of the file:
@@
 Text Label 7800 8150 2    50   ~ 0
 ENC2B
+$Comp
+L kbd:OLED OL?
+U 1 1 6114BDD8
+P 11500 7500
+F 0 "OL?" H 12128 7569 51  0000 L CNN
+F 1 "OLED" H 12128 7479 47  0000 L CNN
+F 2 "" H 11500 7600 60  0001 C CNN
+F 3 "" H 11500 7600 60  0001 C CNN
+	1    11500 7500
+	1    0    0    -1
+$EndComp
+Text GLabel 10750 7400 0    50   Input ~ 0
+i2c_scl
+Text GLabel 10750 7250 0    50   Input ~ 0
+i2c_sda
+$Comp
+L power:GND #PWR?
+U 1 1 6117A46B
+P 10750 7700
+F 0 "#PWR?" H 10750 7450 50  0001 C CNN
+F 1 "GND" H 10755 7527 50  0000 C CNN
+F 2 "" H 10750 7700 50  0001 C CNN
+F 3 "" H 10750 7700 50  0001 C CNN
+	1    10750 7700
+	1    0    0    -1
+$EndComp
+$Comp
+L power:+3.3V #PWR?
+U 1 1 6117B032
+P 10750 7550
+F 0 "#PWR?" H 10750 7400 50  0001 C CNN
+F 1 "+3.3V" H 10765 7723 50  0000 C CNN
+F 2 "" H 10750 7550 50  0001 C CNN
+F 3 "" H 10750 7550 50  0001 C CNN
+	1    10750 7550
+	0    -1   -1   0
+$EndComp
 $EndSCHEMATC

Commit message: finalize unicorn design
Parts:
- added H1, H2, H3, H4, H5, H6, H7: MountingHole, MountingHole:MountingHole_4.5mm, symbol Mechanical:MountingHole
- OL1: renamed from OL?; footprint (none) -> kbd:OLED_v2
Changed lines of the file:
@@
 ENC2B
 $Comp
-L kbd:OLED OL?
+L kbd:OLED OL1
 U 1 1 6114BDD8
 P 11500 7500
-F 0 "OL?" H 12128 7569 51  0000 L CNN
+F 0 "OL1" H 12128 7569 51  0000 L CNN
 F 1 "OLED" H 12128 7479 47  0000 L CNN
-F 2 "" H 11500 7600 60  0001 C CNN
+F 2 "kbd:OLED_v2" H 11500 7600 60  0001 C CNN
 F 3 "" H 11500 7600 60  0001 C CNN
 	1    11500 7500
@@
 i2c_sda
 $Comp
-L power:GND #PWR?
+L power:GND #PWR0103
 U 1 1 6117A46B
 P 10750 7700
-F 0 "#PWR?" H 10750 7450 50  0001 C CNN
+F 0 "#PWR0103" H 10750 7450 50  0001 C CNN
 F 1 "GND" H 10755 7527 50  0000 C CNN
 F 2 "" H 10750 7700 50  0001 C CNN
@@
 $EndComp
 $Comp
-L power:+3.3V #PWR?
+L power:+3.3V #PWR0104
 U 1 1 6117B032
 P 10750 7550
-F 0 "#PWR?" H 10750 7400 50  0001 C CNN
+F 0 "#PWR0104" H 10750 7400 50  0001 C CNN
 F 1 "+3.3V" H 10765 7723 50  0000 C CNN
 F 2 "" H 10750 7550 50  0001 C CNN
@@
 	0    -1   -1   0
 $EndComp
+$Comp
+L Mechanical:MountingHole H1
+U 1 1 6088C715
+P 4550 4600
+F 0 "H1" H 4650 4646 50  0000 L CNN
+F 1 "MountingHole" H 4650 4555 50  0000 L CNN
+F 2 "MountingHole:MountingHole_4.5mm" H 4550 4600 50  0001 C CNN
+F 3 "~" H 4550 4600 50  0001 C CNN
+	1    4550 4600
+	1    0    0    -1
+$EndComp
+$Comp
+L Mechanical:MountingHole H2
+U 1 1 6088D05C
+P 4550 4800
+F 0 "H2" H 4650 4846 50  0000 L CNN
+F 1 "MountingHole" H 4650 4755 50  0000 L CNN
+F 2 "MountingHole:MountingHole_4.5mm" H 4550 4800 50  0001 C CNN
+F 3 "~" H 4550 4800 50  0001 C CNN
+	1    4550 4800
+	1    0    0    -1
+$EndComp
+$Comp
+L Mechanical:MountingHole H3
+U 1 1 6088D61A
+P 4550 5050
+F 0 "H3" H 4650 5096 50  0000 L CNN
+F 1 "MountingHole" H 4650 5005 50  0000 L CNN
+F 2 "MountingHole:MountingHole_4.5mm" H 4550 5050 50  0001 C CNN
+F 3 "~" H 4550 5050 50  0001 C CNN
+	1    4550 5050
+	1    0    0    -1
+$EndComp
+$Comp
+L Mechanical:MountingHole H4
+U 1 1 6088D66C
+P 4550 5250
+F 0 "H4" H 4650 5296 50  0000 L CNN
+F 1 "MountingHole" H 4650 5205 50  0000 L CNN
+F 2 "MountingHole:MountingHole_4.5mm" H 4550 5250 50  0001 C CNN
+F 3 "~" H 4550 5250 50  0001 C CNN
+	1    4550 5250
+	1    0    0    -1
+$EndComp
+$Comp
+L Mechanical:MountingHole H5
+U 1 1 6088D6BE
+P 4550 5450
+F 0 "H5" H 4650 5496 50  0000 L CNN
+F 1 "MountingHole" H 4650 5405 50  0000 L CNN
+F 2 "MountingHole:MountingHole_4.5mm" H 4550 5450 50  0001 C CNN
+F 3 "~" H 4550 5450 50  0001 C CNN
+	1    4550 5450
+	1    0    0    -1
+$EndComp
+$Comp
+L Mechanical:MountingHole H6
+U 1 1 6091BE1F
+P 4550 5700
+F 0 "H6" H 4650 5746 50  0000 L CNN
+F 1 "MountingHole" H 4650 5655 50  0000 L CNN
+F 2 "MountingHole:MountingHole_4.5mm" H 4550 5700 50  0001 C CNN
+F 3 "~" H 4550 5700 50  0001 C CNN
+	1    4550 5700
+	1    0    0    -1
+$EndComp
+$Comp
+L Mechanical:MountingHole H7
+U 1 1 6092BF05
+P 4550 5900
+F 0 "H7" H 4650 5946 50  0000 L CNN
+F 1 "MountingHole" H 4650 5855 50  0000 L CNN
+F 2 "MountingHole:MountingHole_4.5mm" H 4550 5900 50  0001 C CNN
+F 3 "~" H 4550 5900 50  0001 C CNN
+	1    4550 5900
+	1    0    0    -1
+$EndComp
 $EndSCHEMATC

Commit message: add plate and bottom, add rendered images
Parts:
- added BZ1: Buzzer, hy-keebs:Piezo-KLJ-1625, symbol Device:Buzzer
- added D48, D49, D50, D51, D52, D53, D54, D55: WS2812S, LED_SMD:LED_WS2812_PLCC6_5.0x5.0mm_P1.6mm, symbol LED:WS2812S
- U3: footprint breakout_pins:Dual_MCU_QFP_QFN_48_with_breakout_pins -> Package_DFN_QFN:QFN-48-1EP_7x7mm_P0.5mm_EP5.15x5.15mm_ThermalVias
Connections:
- net +3V3: now also D48.3 (VCC), D48.5 (VDD), D49.3 (VCC), D49.5 (VDD), D50.3 (VCC), D50.5 (VDD), D51.3 (VCC), D51.5 (VDD), D52.3 (VCC), D52.5 (VDD), D53.3 (VCC), D53.5 (VDD), D54.3 (VCC), D54.5 (VDD), D55.3 (VCC), D55.5 (VDD)
- net GND: now also D48.6 (VSS), D49.6 (VSS), D50.6 (VSS), D51.6 (VSS), D52.6 (VSS), D53.6 (VSS), D54.6 (VSS), D55.6 (VSS)
- net col10: now also U3.16 (PA6); no longer U3.14 (PA4)
- net col11: now also U3.17 (PA7); no longer U3.15 (PA5)
- net col5: now also U3.34 (PA13); no longer U3.42 (PB6)
- net i2c_scl: now also U3.42 (PB6); no longer U3.21 (PB10)
- net i2c_sda: now also U3.43 (PB7); no longer U3.22 (PB11)
- net LED: now reaches U3.28 (PB15)
- net LED: now also D48.2 (DIN)
- new net: D51.1 (DOUT), D52.2 (DIN)
- new net: D50.1 (DOUT), D51.2 (DIN)
- new net: D52.1 (DOUT), D53.2 (DIN)
- new net: D53.1 (DOUT), D54.2 (DIN)
- new net: D49.1 (DOUT), D50.2 (DIN)
- new net: D54.1 (DOUT), D55.2 (DIN)
- new net: D48.1 (DOUT), D49.2 (DIN)
- new net buzzer_n: BZ1.2 (+), U3.15 (PA5)
- new net buzzer_p: BZ1.1 (-), U3.14 (PA4)
- no-connect marks 9 -> 7

Commit message: Add automation files: now use `make unicorn` or `make unicorn-doc` to generate output and `make clean` to clean up
Parts:
- added R6: 10k, Resistor_SMD:R_0603_1608Metric, symbol Device:R
Connections:
- net +3V3: now also U4.5 (VP); no longer D48.3 (VCC), D48.5 (VDD), D49.3 (VCC), D49.5 (VDD), D50.3 (VCC), D50.5 (VDD), D51.3 (VCC), D51.5 (VDD), D52.3 (VCC), D52.5 (VDD), D53.3 (VCC), D53.5 (VDD), D54.3 (VCC), D54.5 (VDD), D55.3 (VCC), D55.5 (VDD)
- net +5V: now also D48.3 (VCC), D48.5 (VDD), D49.3 (VCC), D49.5 (VDD), D50.3 (VCC), D50.5 (VDD), D51.3 (VCC), D51.5 (VDD), D52.3 (VCC), D52.5 (VDD), D53.3 (VCC), D53.5 (VDD), D54.3 (VCC), D54.5 (VDD), D55.3 (VCC), D55.5 (VDD), R6.1
- net ENC1B: now also U3.22 (PB11); no longer U3.26 (PB13)
- net LED: now also R6.2
- no-connect marks 7 -> 14
Changed lines of the file:
@@
 	1    0    0    -1
 $EndComp
-$Comp
-L power:+3.3V #PWR019
-U 1 1 60789E55
-P 4100 9600
-F 0 "#PWR019" H 4100 9450 50  0001 C CNN
-F 1 "+3.3V" H 4115 9773 50  0000 C CNN
-F 2 "" H 4100 9600 50  0001 C CNN
-F 3 "" H 4100 9600 50  0001 C CNN
-	1    4100 9600
-	1    0    0    -1
-$EndComp
-Wire Wire Line
-	4050 9650 4100 9650
-Wire Wire Line
-	4100 9650 4100 9600
 Wire Wire Line
 	3300 9650 3200 9650
@@
 Text Label 7800 9250 2    50   ~ 0
 ENC1A
-Text Label 7800 9350 2    50   ~ 0
+Text Label 7800 9150 2    50   ~ 0
 ENC1B
 Text Label 7800 8050 2    50   ~ 0
@@
 Wire Wire Line
 	7600 9550 7800 9550
-Text GLabel 8700 4900 0    50   Input ~ 0
+Text GLabel 8100 4900 0    50   Input ~ 0
 LED
-Wire Wire Line
-	8700 4900 8800 4900
 Wire Wire Line
 	9400 4900 9550 4900
@@
 	14000 4900 14100 4900
 NoConn ~ 14700 4900
-$Comp
-L power:+3.3V #PWR0105
-U 1 1 60AECD45
-P 8700 4600
-F 0 "#PWR0105" H 8700 4450 50  0001 C CNN
-F 1 "+3.3V" H 8715 4773 50  0000 C CNN
-F 2 "" H 8700 4600 50  0001 C CNN
-F 3 "" H 8700 4600 50  0001 C CNN
-	1    8700 4600
-	1    0    0    -1
-$EndComp
 Wire Wire Line
 	8700 4600 9000 4600
@@
 Text Label 9100 8550 0    50   ~ 0
 buzzer_n
+NoConn ~ 7800 9350
+$Comp
+L power:+5V #PWR0105
+U 1 1 60906889
+P 8700 4600
+F 0 "#PWR0105" H 8700 4450 50  0001 C CNN
+F 1 "+5V" H 8715 4773 50  0000 C CNN
+F 2 "" H 8700 4600 50  0001 C CNN
+F 3 "" H 8700 4600 50  0001 C CNN
+	1    8700 4600
+	1    0    0    -1
+$EndComp
+$Comp
+L power:+5V #PWR0107
+U 1 1 609429EE
+P 8250 4350
+F 0 "#PWR0107" H 8250 4200 50  0001 C CNN
+F 1 "+5V" H 8265 4523 50  0000 C CNN
+F 2 "" H 8250 4350 50  0001 C CNN
+F 3 "" H 8250 4350 50  0001 C CNN
+	1    8250 4350
+	1    0    0    -1
+$EndComp
+$Comp
+L Device:R R6
+U 1 1 6096D25D
+P 8250 4650
+F 0 "R6" H 8320 4696 50  0000 L CNN
+F 1 "10k" H 8320 4605 50  0000 L CNN
+F 2 "Resistor_SMD:R_0603_1608Metric" V 8180 4650 50  0001 C CNN
+F 3 "" H 8250 4650 50  0001 C CNN
+F 4 "C25804" H 8250 4650 50  0001 C CNN "LCSC Part"
+	1    8250 4650
+	1    0    0    -1
+$EndComp
+Wire Wire Line
+	8100 4900 8250 4900
+Wire Wire Line
+	8250 4800 8250 4900
+Connection ~ 8250 4900
+Wire Wire Line
+	8250 4900 8800 4900
+Wire Wire Line
+	8250 4500 8250 4350
+$Comp
+L power:+3.3V #PWR05
+U 1 1 60A58ADD
+P 4300 9450
+F 0 "#PWR05" H 4300 9300 50  0001 C CNN
+F 1 "+3.3V" H 4315 9623 50  0000 C CNN
+F 2 "" H 4300 9450 50  0001 C CNN
+F 3 "" H 4300 9450 50  0001 C CNN
+	1    4300 9450
+	1    0    0    -1
+$EndComp
+Wire Wire Line
+	4300 9450 4300 9650
+$Comp
+L power:GND #PWR0108
+U 1 1 60B051BC
+P 8950 10500
+F 0 "#PWR0108" H 8950 10250 50  0001 C CNN
+F 1 "GND" H 8955 10327 50  0000 C CNN
+F 2 "" H 8950 10500 50  0001 C CNN
+F 3 "" H 8950 10500 50  0001 C CNN
+	1    8950 10500
+	1    0    0    -1
+$EndComp
+$Comp
+L power:+5V #PWR0110
+U 1 1 60B0722C
+P 9850 10500
+F 0 "#PWR0110" H 9850 10350 50  0001 C CNN
+F 1 "+5V" H 9865 10673 50  0000 C CNN
+F 2 "" H 9850 10500 50  0001 C CNN
+F 3 "" H 9850 10500 50  0001 C CNN
+	1    9850 10500
+	-1   0    0    1
+$EndComp
+$Comp
+L power:PWR_FLAG #FLG0102
+U 1 1 60B09274
+P 9850 10500
+F 0 "#FLG0102" H 9850 10575 50  0001 C CNN
+F 1 "PWR_FLAG" H 9850 10673 50  0000 C CNN
+F 2 "" H 9850 10500 50  0001 C CNN
+F 3 "" H 9850 10500 50  0001 C CNN
+	1    9850 10500
+	1    0    0    -1
+$EndComp
+NoConn ~ 7800 7350
+NoConn ~ 7800 7450
+NoConn ~ 7800 7650
+NoConn ~ 7800 7750
+NoConn ~ 7800 7850
+NoConn ~ 7800 9050
 $EndSCHEMATC

Commit message: route pcb with new pin assginments, add bridges for led, add test points
Parts:
- added 3V3, 5V1, BOOT0, GND1, GND2, NRST1: TestPoint, TestPoint:TestPoint_THTPad_D1.5mm_Drill0.7mm, symbol Connector:TestPoint
- added JP1, JP2: SolderJumper_2_Open, Jumper:SolderJumper-2_P1.3mm_Open_TrianglePad1.0x1.5mm, symbol Jumper:SolderJumper_2_Open
- added R9: 0, Resistor_SMD:R_0603_1608Metric, symbol Device:R
Connections:
- net +3V3: now also 3V3.1
- net +5V: now also 5V1.1
- net BOOT0: now also BOOT0.1
- net GND: now also BZ1.2 (+), GND1.1, GND2.1
- net LED: now also JP1.2 (B), JP2.2 (B), R9.1; no longer U3.28 (PB15)
- net NRST: now also NRST1.1
- net buzzer_p: now also U3.29 (PA8); no longer U3.14 (PA4)
- net col2: now also U3.26 (PB13); no longer U3.39 (PB3)
- net col3: now also U3.27 (PB14); no longer U3.40 (PB4)
- net col4: now also U3.28 (PB15); no longer U3.41 (PB5)
- net row2: now also U3.31 (PA10); no longer U3.30 (PA9)
- net row3: now also U3.30 (PA9); no longer U3.29 (PA8)
- net buzzer_n: no longer names the net of U3.15 (PA5)
- net buzzer_n: no longer BZ1.2 (+)
- new net LED_PWM: JP2.1 (A), R9.2, U3.40 (PB4)
- new net LED_SPI: JP1.1 (A), U3.41 (PB5)
Changed lines of the file:
@@
 	1    0    0    -1
 $EndComp
-Text Label 7800 8450 2    50   ~ 0
+Text Label 7800 9450 2    50   ~ 0
 col3
-Text Label 7800 8550 2    50   ~ 0
+Text Label 7800 9550 2    50   ~ 0
 col4
 Text Label 9100 9350 0    50   ~ 0
@@
 Wire Wire Line
 	7800 7150 7550 7150
-NoConn ~ 9100 9050
-NoConn ~ 7800 8250
-NoConn ~ 7800 9450
-Text Label 9100 8850 0    50   ~ 0
+Text Label 9100 8950 0    50   ~ 0
 row3
 Wire Wire Line
@@
 Connection ~ 5350 3700
 Connection ~ 7850 3700
-Text Label 7800 8350 2    50   ~ 0
+Text Label 7800 9350 2    50   ~ 0
 col2
 Text Label 9100 9550 0    50   ~ 0
@@
 Text Label 9100 9450 0    50   ~ 0
 col0
-Text Label 9100 8950 0    50   ~ 0
+Text Label 9100 9050 0    50   ~ 0
 row2
 Text Label 7800 8850 2    50   ~ 0
@@
 	1    0    0    -1
 $EndComp
-Text GLabel 7600 9550 0    50   Input ~ 0
-LED
-Wire Wire Line
-	7600 9550 7800 9550
+Text GLabel 7600 8450 0    50   Input ~ 0
+LED_PWM
+Wire Wire Line
+	7600 8450 7800 8450
 Text GLabel 8100 4900 0    50   Input ~ 0
 LED
@@
 Text Label 11500 9100 2    50   ~ 0
 buzzer_n
-Text Label 9100 8450 0    50   ~ 0
+Text Label 9100 8850 0    50   ~ 0
 buzzer_p
-Text Label 9100 8550 0    50   ~ 0
+Text Label 10650 9100 0    50   ~ 0
 buzzer_n
-NoConn ~ 7800 9350
 $Comp
 L power:+5V #PWR0105
@@
 NoConn ~ 7800 7850
 NoConn ~ 7800 9050
+$Comp
+L power:GND #PWR0109
+U 1 1 609AC589
+P 10650 9300
+F 0 "#PWR0109" H 10650 9050 50  0001 C CNN
+F 1 "GND" H 10655 9127 50  0000 C CNN
+F 2 "" H 10650 9300 50  0001 C CNN
+F 3 "" H 10650 9300 50  0001 C CNN
+	1    10650 9300
+	1    0    0    -1
+$EndComp
+Wire Wire Line
+	10650 9100 10650 9300
+NoConn ~ 7800 8350
+NoConn ~ 7800 8250
+NoConn ~ 9100 8450
+NoConn ~ 9100 8550
+$Comp
+L Jumper:SolderJumper_2_Open JP1
+U 1 1 60B178A8
+P 7000 4300
+F 0 "JP1" H 7000 4505 50  0000 C CNN
+F 1 "SolderJumper_2_Open" H 7000 4414 50  0000 C CNN
+F 2 "Jumper:SolderJumper-2_P1.3mm_Open_TrianglePad1.0x1.5mm" H 7000 4300 50  0001 C CNN
+F 3 "~" H 7000 4300 50  0001 C CNN
+	1    7000 4300
+	1    0    0    -1
+$EndComp
+Text GLabel 7600 8550 0    50   Input ~ 0
+LED_SPI
+Wire Wire Line
+	7600 8550 7800 8550
+Text GLabel 6700 4650 0    50   Input ~ 0
+LED_PWM
+Text GLabel 6700 4300 0    50   Input ~ 0
+LED_SPI
+Wire Wire Line
+	6700 4300 6850 4300
+Wire Wire Line
+	6700 4650 6850 4650
+Text GLabel 7550 4300 2    50   Input ~ 0
+LED
+Wire Wire Line
+	7150 4300 7400 4300
+Wire Wire Line
+	7400 4300 7400 4650
+Wire Wire Line
+	7400 4650 7150 4650
+Connection ~ 7400 4300
+Wire Wire Line
+	7400 4300 7550 4300
+$Comp
+L Jumper:SolderJumper_2_Open JP2
+U 1 1 60C4E8D0
+P 7000 4650
+F 0 "JP2" H 7000 4855 50  0000 C CNN
+F 1 "SolderJumper_2_Open" H 7000 4764 50  0000 C CNN
+F 2 "Jumper:SolderJumper-2_P1.3mm_Open_TrianglePad1.0x1.5mm" H 7000 4650 50  0001 C CNN
+F 3 "~" H 7000 4650 50  0001 C CNN
+	1    7000 4650
+	1    0    0    -1
+$EndComp
+$Comp
+L Device:R R9
+U 1 1 60C512C1
+P 7000 4900
+F 0 "R9" H 7070 4946 50  0000 L CNN
+F 1 "0" H 7070 4855 50  0000 L CNN
+F 2 "Resistor_SMD:R_0603_1608Metric" V 6930 4900 50  0001 C CNN
+F 3 "" H 7000 4900 50  0001 C CNN
+F 4 "C21189" H 7000 4900 50  0001 C CNN "LCSC Part"
+	1    7000 4900
+	0    1    1    0
+$EndComp
+Text GLabel 6700 4900 0    50   Input ~ 0
+LED_PWM
+Wire Wire Line
+	6700 4900 6850 4900
+Wire Wire Line
+	7150 4900 7400 4900
+Wire Wire Line
+	7400 4900 7400 4650
+Connection ~ 7400 4650
+$Comp
+L Connector:TestPoint NRST1
+U 1 1 60CC3A36
+P 13650 6100
+F 0 "NRST1" H 13592 6126 50  0000 R CNN
+F 1 "TestPoint" H 13592 6217 50  0000 R CNN
+F 2 "TestPoint:TestPoint_THTPad_D1.5mm_Drill0.7mm" H 13850 6100 50  0001 C CNN
+F 3 "" H 13850 6100 50  0001 C CNN
+	1    13650 6100
+	-1   0    0    1
+$EndComp
+Text GLabel 13400 6000 1    50   Input ~ 0
+BOOT0
+Text GLabel 13650 6000 1    50   Input ~ 0
+NRST
+$Comp
+L power:+3.3V #PWR09
+U 1 1 60D29157
+P 13950 5950
+F 0 "#PWR09" H 13950 5800 50  0001 C CNN
+F 1 "+3.3V" H 13965 6123 50  0000 C CNN
+F 2 "" H 13950 5950 50  0001 C CNN
+F 3 "" H 13950 5950 50  0001 C CNN
+	1    13950 5950
+	1    0    0    -1
+$EndComp
+$Comp
+L power:+5V #PWR012
+U 1 1 60D2A5AB
+P 14250 5950
+F 0 "#PWR012" H 14250 5800 50  0001 C CNN
+F 1 "+5V" H 14265 6123 50  0000 C CNN
+F 2 "" H 14250 5950 50  0001 C CNN
+F 3 "" H 14250 5950 50  0001 C CNN
+	1    14250 5950
+	1    0    0    -1
+$EndComp
+$Comp
+L power:GND #PWR013
+U 1 1 60D2B5E2
+P 14500 5950
+F 0 "#PWR013" H 14500 5700 50  0001 C CNN
+F 1 "GND" H 14505 5777 50  0000 C CNN
+F 2 "" H 14500 5950 50  0001 C CNN
+F 3 "" H 14500 5950 50  0001 C CNN
+	1    14500 5950
+	-1   0    0    1
+$EndComp
+$Comp
+L Connector:TestPoint BOOT0
+U 1 1 60D2C9A6
+P 13400 6100
+F 0 "BOOT0" H 13342 6126 50  0000 R CNN
+F 1 "TestPoint" H 13342 6217 50  0000 R CNN
+F 2 "TestPoint:TestPoint_THTPad_D1.5mm_Drill0.7mm" H 13600 6100 50  0001 C CNN
+F 3 "" H 13600 6100 50  0001 C CNN
+	1    13400 6100
+	-1   0    0    1
+$EndComp
+$Comp
+L Connector:TestPoint 3V3
+U 1 1 60D2CD80
+P 13950 6100
+F 0 "3V3" H 13892 6126 50  0000 R CNN
+F 1 "TestPoint" H 13892 6217 50  0000 R CNN
+F 2 "TestPoint:TestPoint_THTPad_D1.5mm_Drill0.7mm" H 14150 6100 50  0001 C CNN
+F 3 "" H 14150 6100 50  0001 C CNN
+	1    13950 6100
+	-1   0    0    1
+$EndComp
+$Comp
+L Connector:TestPoint 5V1
+U 1 1 60D2D3F8
+P 14250 6100
+F 0 "5V1" H 14192 6126 50  0000 R CNN
+F 1 "TestPoint" H 14192 6217 50  0000 R CNN
+F 2 "TestPoint:TestPoint_THTPad_D1.5mm_Drill0.7mm" H 14450 6100 50  0001 C CNN
+F 3 "" H 14450 6100 50  0001 C CNN
+	1    14250 6100
+	-1   0    0    1
+$EndComp
+$Comp
+L Connector:TestPoint GND1
+U 1 1 60D2D866
+P 14500 6100
+F 0 "GND1" H 14442 6126 50  0000 R CNN
+F 1 "TestPoint" H 14442 6217 50  0000 R CNN
+F 2 "TestPoint:TestPoint_THTPad_D1.5mm_Drill0.7mm" H 14700 6100 50  0001 C CNN
+F 3 "" H 14700 6100 50  0001 C CNN
+	1    14500 6100
+	-1   0    0    1
+$EndComp
+Wire Wire Line
+	13400 6000 13400 6100
+Wire Wire Line
+	13650 6000 13650 6100
+Wire Wire Line
+	13950 5950 13950 6100
+Wire Wire Line
+	14250 5950 14250 6100
+Wire Wire Line
+	14500 5950 14500 6100
+$Comp
+L Connector:TestPoint GND2
+U 1 1 60E2F852
+P 14950 6100
+F 0 "GND2" H 14892 6126 50  0000 R CNN
+F 1 "TestPoint" H 14892 6217 50  0000 R CNN
+F 2 "TestPoint:TestPoint_THTPad_D1.5mm_Drill0.7mm" H 15150 6100 50  0001 C CNN
+F 3 "" H 15150 6100 50  0001 C CNN
+	1    14950 6100
+	-1   0    0    1
+$EndComp
+$Comp
+L power:GND #PWR0111
+U 1 1 60E2FEB7
+P 14950 5950
+F 0 "#PWR0111" H 14950 5700 50  0001 C CNN
+F 1 "GND" H 14955 5777 50  0000 C CNN
+F 2 "" H 14950 5950 50  0001 C CNN
+F 3 "" H 14950 5950 50  0001 C CNN
+	1    14950 5950
+	-1   0    0    1
+$EndComp
+Wire Wire Line
+	14950 5950 14950 6100
 $EndSCHEMATC

Commit message: use f411 mcu
Parts:
- removed U3: STM32F072CBUx, Package_DFN_QFN:QFN-48-1EP_7x7mm_P0.5mm_EP5.15x5.15mm_ThermalVias, symbol MCU_ST_STM32F0:STM32F072CBUx
- added C14, C15: 0.1uF, Capacitor_SMD:C_0603_1608Metric, symbol Device:C
- added C16: 1.5pF, Capacitor_SMD:C_0603_1608Metric, symbol Device:C
- added C7, C8: 20pF, Capacitor_SMD:C_0603_1608Metric, symbol Device:C
- added J1, J3: Conn_01x06, Connector_PinHeader_2.54mm:PinHeader_1x06_P2.54mm_Vertical, symbol Connector_Generic:Conn_01x06
- added J4, J5, J6: Conn_01x04, Connector_PinHeader_2.54mm:PinHeader_1x04_P2.54mm_Vertical, symbol Connector_Generic:Conn_01x04
- added U2: STM32F411CCUx, Package_DFN_QFN:QFN-48-1EP_7x7mm_P0.5mm_EP5.6x5.6mm, symbol MCU_ST_STM32F4:STM32F411CCUx
- added Y1: 25M Hz, Crystal:Crystal_SMD_3225-4Pin_3.2x2.5mm, symbol Device:Crystal_GND24
- added Y2: 32.768KHz, Crystal:Crystal_SMD_3215-2Pin_3.2x1.5mm, symbol Device:Crystal
- C11: Field6 (none) -> ESR < 1Ohm
- C9: value 4.7uF -> 1.5pF; Field4 0603 -> (none); LCSC Part C19666 -> C1639
- TP1: renamed from BOOT0; value TestPoint -> BOOT0
- TP2: renamed from NRST1; value TestPoint -> NRST
- TP3: renamed from 3V3; value TestPoint -> 3V3
- TP4: renamed from 5V1; value TestPoint -> 5V
- TP5: renamed from GND1; value TestPoint -> GND
- TP6: renamed from GND2; value TestPoint -> GND
Connections:
- net +3V3: now also C10.1, C6.1, C14.1, C15.1, J6.1 (Pin_1), U2.1 (VBAT), U2.24 (VDD), U2.36 (VDD), U2.48 (VDD), U2.9 (VDDA); no longer C10.2, C11.2, C6.2, C9.1
- net BOOT0: now also U2.44 (BOOT0)
- net D+: now also U2.33 (PA12)
- net D-: now also U2.32 (PA11)
- net ENC1A: now also U2.25 (PB12)
- net ENC1B: now also U2.21 (PB10)
- net ENC2A: now also U2.18 (PB0)
- net ENC2B: now also U2.20 (PB2)
- net GND: now also C10.2, C6.2, C14.2, C15.2, C16.2, C7.2, C8.2, J6.4 (Pin_4), U2.23 (VSS), U2.35 (VSS), U2.47 (VSS), U2.49 (VSS), U2.8 (VSSA), Y1.2, Y1.4; no longer C10.1, C6.1
- net LED_PWM: now also U2.19 (PB1)
- net LED_SPI: now also U2.41 (PB5)
- net NRST: now also U2.7 (NRST)
- net buzzer_p: now also U2.29 (PA8)
- net col1: now also J1.2 (Pin_2), U2.38 (PA15)
- net col10: now also J3.5 (Pin_5), U2.16 (PA6)
- net col11: now also J3.6 (Pin_6), U2.17 (PA7)
- net col2: now also J1.3 (Pin_3), U2.26 (PB13)
- net col3: now also J1.4 (Pin_4), U2.27 (PB14)
- net col4: now also J1.5 (Pin_5), U2.28 (PB15)
- net col6: now also J3.1 (Pin_1), U2.10 (PA0)
- net col7: now also J3.2 (Pin_2), U2.11 (PA1)
- net col8: now also J3.3 (Pin_3), U2.12 (PA2)
- net col9: now also J3.4 (Pin_4), U2.13 (PA3)
- net i2c_scl: now also U2.42 (PB6)
- net i2c_sda: now also U2.43 (PB7)
- net row0: now also J4.1 (Pin_1), J5.1 (Pin_1), U2.46 (PB9)
- net row1: now also J4.2 (Pin_2), J5.2 (Pin_2), U2.45 (PB8)
- net row2: now also J4.3 (Pin_3), J5.3 (Pin_3), U2.31 (PA10)
- net row3: now also J4.4 (Pin_4), J5.4 (Pin_4), U2.30 (PA9)
- net col0 renamed SWCLK
- net SWCLK: now also J1.1 (Pin_1), J6.2 (Pin_2), U2.37 (PA14)
- net col5 renamed SWDIO
- net SWDIO: now also J1.6 (Pin_6), J6.3 (Pin_3), U2.34 (PA13)
- new net: C9.1, U2.3 (PC14), Y2.1
- new net: C16.1, U2.4 (PC15), Y2.2
- new net: C7.1, U2.5 (PH0), Y1.1
- new net: C8.1, U2.6 (PH1), Y1.3
- new net VCAP1: C11.2, U2.22 (VCAP1)
- no-connect marks 14 -> 9
Other:
- moved on the sheet: BZ1, C10, C11, C12, C13, C5, C6, OL1
