File: unicorn-mx/unicorn/unicorn.kicad_pcb (KiCad board)
At the start: 2 copper layers, 268.2 x 110.5 mm, 145 parts, among them J2 USB_C, K1 KEYSW, K10 KEYSW, K11 KEYSW, K12 KEYSW, K13 KEYSW, K14 KEYSW, K15 KEYSW, K16 KEYSW, K17 KEYSW, K18 KEYSW, K19 KEYSW, K2 KEYSW, K20 KEYSW, K21 KEYSW, K22 KEYSW, K23 KEYSW, K24 KEYSW, K25 KEYSW, K26 KEYSW, K27 KEYSW, K28 KEYSW, K29 KEYSW, K3 KEYSW, K30 KEYSW, K31 KEYSW, K32 KEYSW, K33 KEYSW, K34 KEYSW, K35 KEYSW, K36 KEYSW, K37 KEYSW, K38 KEYSW, K39 KEYSW, K4 KEYSW, K40 KEYSW, K41 KEYSW, K42 KEYSW, K43 KEYSW, K44 KEYSW, K5 KEYSW, K6 KEYSW, K7 KEYSW, K8 KEYSW, K9 KEYSW, Q1 MMBT3904, SW1 SW_Push, SW2 Rotary_Encoder_Switch, SW3 Rotary_Encoder_Switch, U1 XC6206PxxxMR, U3 STM32F072CBUx, U4 SRV05-4

Commit message: use f411 mcu
Parts:
- removed U3: STM32F072CBUx, Package_DFN_QFN:QFN-48-1EP_7x7mm_P0.5mm_EP5.15x5.15mm_ThermalVias
- added C14: 0.1uF, Capacitor_SMD:C_0603_1608Metric, B.Cu at (146.5, 74.2)
- added C15: 0.1uF, Capacitor_SMD:C_0603_1608Metric, B.Cu at (156.0, 91.0)
- added C16: 1.5pF, Capacitor_SMD:C_0603_1608Metric, B.Cu at (157.4, 75.3)
- added C7: 20pF, Capacitor_SMD:C_0603_1608Metric, B.Cu at (161.6, 74.0)
- added C8: 20pF, Capacitor_SMD:C_0603_1608Metric, B.Cu at (166.8, 74.0)
- added J1: Conn_01x06, Connector_PinHeader_2.54mm:PinHeader_1x06_P2.54mm_Vertical, F.Cu at (35.9, 100.5)
- added J3: Conn_01x06, Connector_PinHeader_2.54mm:PinHeader_1x06_P2.54mm_Vertical, F.Cu at (258.3, 100.5)
- added J4: Conn_01x04, Connector_PinHeader_2.54mm:PinHeader_1x04_P2.54mm_Vertical, F.Cu at (31.2, 85.4)
- added J5: Conn_01x04, Connector_PinHeader_2.54mm:PinHeader_1x04_P2.54mm_Vertical, F.Cu at (276.9, 84.7)
- added J6: Conn_01x04, Connector_PinHeader_2.54mm:PinHeader_1x04_P2.54mm_Vertical, F.Cu at (165.2, 130.8)
- added U2: STM32F411CCUx, Package_DFN_QFN:QFN-48-1EP_7x7mm_P0.5mm_EP5.6x5.6mm, B.Cu at (154.5, 80.7)
- added Y1: 25M, Crystal:Crystal_SMD_3225-4Pin_3.2x2.5mm, B.Cu at (164.3, 74.1)
- added Y2: 32.768KHz, Crystal:Crystal_SMD_3215-2Pin_3.2x1.5mm, B.Cu at (157.8, 73.1)
- C9: value 4.7uF -> 1.5pF
- TP1: renamed from BOOT0; value TestPoint -> BOOT0
- TP2: renamed from NRST1; value TestPoint -> NRST
- TP3: renamed from 3V3; value TestPoint -> 3V3
- TP4: renamed from 5V1; value TestPoint -> 5V
- TP5: renamed from GND1; value TestPoint -> GND
- TP6: renamed from GND2; value TestPoint -> GND
- moved C5 16.1 mm to (148.0, 71.8), turned to 180 degrees
- moved C9 7.16 mm to (154.9, 73.2), turned to 270 degrees
- moved C10 5.28 mm to (167.0, 77.1)
- moved R9 4.98 mm to (121.0, 100.3)
- moved C11 1.61 mm to (158.3, 90.4), turned to 90 degrees
- turned C6 to 270 degrees
Connections:
- net /col0 renamed /SWCLK
- net /col5 renamed /SWDIO
- C10 pad 1: GND -> +3V3
- C10 pad 2: +3V3 -> GND
- C11 pad 2: +3V3 -> /VCAP1
- C6 pad 1: GND -> +3V3
- C6 pad 2: +3V3 -> GND
- C9 pad 1: +3V3 -> Net-(C9-Pad1)
Routing:
- net /col8: track 124.0 -> 311.3 mm, vias 6 -> 9
- net /SWDIO: track 130.7 -> 285.2 mm, vias 6 -> 8
- net /row3: track 173.0 -> 319.9 mm, vias 2 -> 4
- net /row0: track 249.9 -> 376.4 mm, vias 2 -> 4
- net /SWCLK: track 174.1 -> 289.3 mm, vias 0 -> 3
- net /col6: track 87.3 -> 194.9 mm, vias 4 -> 6
- net /row1: track 269.0 -> 351.3 mm, vias 2 -> 4
- net /col7: track 109.7 -> 190.6 mm
- net /row2: track 257.8 -> 332.7 mm, vias 2 -> 5
- net /col4: track 147.6 -> 212.4 mm, vias 6 -> 7
- net /col3: track 177.2 -> 235.1 mm, vias 6 -> 7
- net /col9: track 157.8 -> 192.5 mm
- net /col10: track 144.7 -> 177.8 mm, vias 5 -> 6
- net /col2: track 197.5 -> 228.8 mm
- net /col1: track 166.2 -> 196.2 mm
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Other:
- board text added: "0 1 2 3"
- board text added: "0 1 2 3 4 5 6"
- board text added: "3V3"
- board text added: "5V"
- board text added: "6 7 8 9 10 11"
- board text added: "BOOT0"
- board text added: "GND"
- board text added: "NRST"
- board text added: "SWC"
- board text added: "SWD"
- board text added: "col"
- board text added: "row"

Commit message: Add back rotation for jlcpcb positions, as most footproints still needs rotation.
Parts:
- Y1: value 25M -> 25MHz
